File: op-amp/op-amp_reverb_driver.kicad_pcb (KiCad board)
At the start: 2 copper layers, 109 x 64.5 mm, 80 parts, among them J1 AC IN, J10 Audio Out, J2 From Tank, J3 Audio In, J4 Dry Level, J5 power led, J6 Mute, J7 Reverb Level, J8 Power, J9 To Tank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

Commit message: at a natural point of fail
Parts:
- D9, R9: moved to B.Cu
- F1: footprint footprints:Fuseholder5x20_horiz_open_lateral_Type-II -> Fuse_Holders_and_Fuses:Fuseholder5x20_horiz_open_lateral_Type-II
- T1: footprint Transformers:Hammond_229_series_low_profile_transformers -> Transformer_THT:Transformer_Hammond_229B34
- moved R9 6.61 mm to (37.1, 112.2), turned to 0 degrees
- moved D9 5.33 mm to (34.0, 112.2), turned to 180 degrees
- moved F1 4.47 mm to (25.1, 74.2)
- moved J1 2.91 mm to (26.9, 99.8)
Connections:
- net /AC_L renamed /Sheet5FCCC7F5/AC_L
- net /AC_N renamed /Sheet5FCCC7F5/AC_N
- Q1 pad 1: Net-(C13-Pad1) -> Net-(Q1-Pad1)
- Q1 pad 3: Net-(Q1-Pad3) -> Net-(C13-Pad1)
- Q2 pad 1: Net-(C13-Pad2) -> Net-(Q2-Pad1)
- Q2 pad 2: Net-(Q2-Pad2) -> /-15V
- Q2 pad 3: /-15V -> Net-(C13-Pad2)
- R16 pad 1: Net-(Q1-Pad3) -> Net-(Q1-Pad1)
- R17 pad 2: Net-(Q2-Pad2) -> Net-(Q2-Pad1)
Routing:
- net /-15V: track 190.5 -> 207.4 mm
- net Net-(Q1-Pad1): track 0.00 -> 8.10 mm, vias 0 -> 1
- net Net-(C13-Pad1): track 16.8 -> 24.9 mm
- net Net-(C12-Pad2): track 151.6 -> 145.2 mm, vias 6 -> 5
- net Net-(Q2-Pad1): track 0.00 -> 4.68 mm
- net Net-(C11-Pad1): track 112.9 -> 108.6 mm, vias 5 -> 6
- net /Sheet5FCCC7F5/AC_N: track 68.5 -> 72.3 mm
- net Net-(Q2-Pad2): track 3.58 -> 0.00 mm
- net Net-(Q1-Pad3): track 3.18 -> 0.00 mm
- net Earth: track 47.6 -> 50.1 mm, vias 23 -> 26
- net Net-(F1-Pad1): track 59.4 -> 57.5 mm
- net Net-(D9-Pad1): track 2.46 -> 1.45 mm
- net /Sheet5FCCC7F5/AC_L: track 14.1 -> 13.5 mm
