File: op-amp/op-amp_reverb_driver.sch (KiCad schematic (older format))
At the start: 80 parts, among them J1 AC IN, J2 From Tank, J3 Audio In, J4 Dry Level, J5 power led, J6 Mute, J7 Reverb Level, J8 Power, J9 To Tank, Q1 BD139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

Commit message: lay out the PCB and submit it to OSHPark
Parts:
- J10: renamed from Output1; value To Tank -> Audio Out
- U3, U4: footprint Package_TO_SOT_SMD:TO-252-3_TabPin2 -> Package_TO_SOT_SMD:TO-252-2
Connections:
- net Earth: now also C21.2, C22.1
- net INPUT: no longer names the net of J3.1 (Pin_1), R2.2
Other:
- moved on the sheet: C11, C12, C14, C15, C16, C17, C18, C19, C21, C22, C23, C24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

Commit message: at a natural point of fail
Parts:
- removed C11, C12, C16, C17, C18, C19, C23, C24: 0.1uF, Capacitor_SMD:C_0603_1608Metric, symbol Device:C
- removed C14, C15: 10uF, Capacitor_SMD:C_0805_2012Metric, symbol Device:C_Polarized
- removed C21, C22: 100uF, Capacitor_SMD:CP_Elec_8x10.5, symbol Device:C_Polarized
- removed C3, C4: 3000uF, Capacitor_SMD:CP_Elec_18x22, symbol Device:C_Polarized
- removed D1, D2, D3, D4, D5, D6, D7, D8: MBRD6100CTTR, Package_TO_SOT_SMD:TO-252-2, symbol Diode:MBRD6100CTTR
- removed D9: LED, Diode_SMD:D_0603_1608Metric, symbol Device:LED
- removed F1: 1A, footprints:Fuseholder5x20_horiz_open_lateral_Type-II, symbol Device:Fuse
- removed J1: AC IN, Connector_Terminal_Block:TerminalBlock-3_P5.08mm, symbol Connector:Screw_Terminal_01x03
- removed J5: power led, Connector_Terminal_Block:TerminalBlock_1x02_P2.54mm_Horizontal, symbol Connector:Screw_Terminal_01x02
- removed J8: Power, Connector_Terminal_Block:TerminalBlock_1x03_P2.54mm_Horizontal, symbol Connector:Screw_Terminal_01x03
- removed R9: 10K, Resistor_SMD:R_0603_1608Metric, symbol Device:R
- removed T1: Hammond_229B34, Transformers:Hammond_229_series_low_profile_transformers, symbol local:Hammond_229B34
- removed unit 3 of U1
- removed unit 3 of U2
- removed U3: L7815, Package_TO_SOT_SMD:TO-252-2, symbol Regulator_Linear:L7815
- removed U4: L7915, Package_TO_SOT_SMD:TO-252-2, symbol Regulator_Linear:L7915
- R14, R15: value 3.9K -> 4.7K
Connections:
- net -15V: now also Q2.2 (C); no longer Q2.1 (E)
- net at R17.2: now also Q2.1 (E); no longer Q2.2 (C)
Other:
- moved on the sheet: C1, C10, C13, C2, C20, C5, C6, C7, C8, C9, D10, D11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
